Commit message: add dino

File: awd/data/assets/dino/dino.urdf (robot description, URDF)
Before this commit: robot eyecandy, 54 links, 53 joints
Links:
- link right_roll_to_pitch: mass 0.0276699 -> 0.059066
- link tail_connector: mass 1e-09 -> 0.00399713
Joints:
- joint act_in_hip_left: origin xyz=0.0323698 0.01025 0.00236 rpy=3.14159 1.5708 0 -> xyz=0.0523698 0.01025 0.00236 rpy=-3.14159 1.5708 0
- joint act_in_hip_rtop: origin xyz=-0.0323698 -0.01025 0.00236 rpy=1.09839e-16 1.5708 0 -> xyz=-0.0523698 -0.01025 0.00236 rpy=1.09839e-16 1.5708 0
- joint cover_to_leg_left: origin xyz=-0.007 -0.02 -0.01 rpy=-4.37442e-16 1.30809e-16 -2.30383 -> xyz=-0.007 -0.02 -0.01 rpy=-2.51562e-14 -3.1562e-15 -2.30383
- joint foot_3: origin xyz=-0.0563458 0.0580779 0.017 rpy=-3.14159 9.11218e-16 -0.349066 -> xyz=-0.0563458 0.0580779 0.017 rpy=-3.14159 3.67918e-16 -0.349066
- joint foot_4: origin xyz=-0.00544005 0.0390203 0.00657843 rpy=1.5708 -2.52241e-16 -0.386778 -> xyz=-0.00544005 0.0390203 0.00657843 rpy=1.5708 -1.04558e-16 -0.386778
- joint left_act_shin: origin xyz=0.00337105 0.0348373 -0.005 rpy=-3.14159 -5.93561e-16 -1.6057 -> xyz=0.00337105 0.0348373 -0.005 rpy=-3.14159 3.36129e-15 -1.6057
- joint left_ankle: origin xyz=-0.03275 0.01025 -0.03505 rpy=-5.19692e-16 1.33974e-14 1.5708 -> xyz=-0.03275 0.01025 -0.03505 rpy=2.29827e-15 1.50863e-15 1.5708
- joint left_foot_frame: origin xyz=-0.0138727 0.005 -0.00631827 rpy=-1.23601e-30 -0.025933 3.14159 -> xyz=-0.0138727 0.005 -0.00631827 rpy=-1.11449e-16 -0.025933 3.14159
- joint left_hip_pitch: origin xyz=-0.03275 0.01025 -0.03505 rpy=3.62855e-32 2.5326e-32 -0.523599 -> xyz=-0.03275 0.01025 -0.03505 rpy=-1.67045e-31 1.10934e-31 -0.523599
- joint left_hip_roll: origin xyz=0.01905 -3.08781e-16 -0.046015 rpy=-1.5708 -3.98119e-16 1.5708 -> xyz=0.01905 2.13718e-15 -0.046015 rpy=-1.5708 2.10942e-15 1.5708
- joint left_hip_yaw: origin xyz=-0.03275 -0.01025 -0.03505 rpy=1.22125e-15 1.65811e-16 3.14159 -> xyz=-0.03275 -0.01025 -0.03505 rpy=1.22125e-15 -3.35143e-29 3.14159
- joint left_knee: origin xyz=0.0340323 -0.0044073 -0.03505 rpy=1.13912e-16 4.15533e-17 -2.44346 -> xyz=0.0340323 -0.0044073 -0.03505 rpy=-3.90287e-16 -1.12803e-15 -2.44346
- joint leg_act_left: origin xyz=-0.00580147 -0.0504366 -0.006 rpy=-3.14159 -1.07236e-16 -1.5708 -> xyz=-0.00580147 -0.0504366 -0.006 rpy=3.14159 2.54608e-16 -1.5708
- joint right_hip_roll: origin xyz=0.01905 1.66533e-16 -0.046015 rpy=-1.5708 5.52966e-16 1.5708 -> xyz=0.01905 -2.77556e-17 -0.046015 rpy=-1.5708 5.52966e-16 1.5708

Commit message: dino final urdf working

File: awd/data/assets/dino/dino.urdf (robot description, URDF)
Before this commit: robot eyecandy, 54 links, 53 joints
Links:
- link body_back: mass 0.313965 -> 0.310516
- link body_front: mass 0.156983 -> 0.153978
Joints:
- removed joint act_in_hip_rtop
- added joint act_in_hip_right: type fixed, parent right_roll_to_pitch, child actuator_6, origin xyz=-0.0523698 -0.01025 0.00236 rpy=-1.80411e-16 1.5708 0, axis 0 0 1, limit effort=10 velocity=10
- joint act_in_hip_left: origin xyz=0.0523698 0.01025 0.00236 rpy=-3.14159 1.5708 0 -> xyz=0.0523698 0.01025 0.00236 rpy=3.14159 1.5708 0
- joint cover_to_leg_left: origin xyz=-0.007 -0.02 -0.01 rpy=-2.51562e-14 -3.1562e-15 -2.30383 -> xyz=-0.007 -0.02 -0.01 rpy=-6.58031e-17 -6.41721e-17 -2.30383
- joint cover_to_leg_right: origin xyz=0.0138205 0.0160622 -0.01 rpy=-1.47478e-15 -2.43254e-15 1.309 -> xyz=-0.007 0.02 -0.01 rpy=1.73993e-16 5.2061e-16 2.35619
- joint foot_1: origin xyz=-0.0194157 -0.0373546 0.017 rpy=3.14159 -2.63189e-16 0.436332 -> xyz=-0.0256494 0.0333834 0.017 rpy=-3.14159 1.11474e-15 -1.5708
- joint foot_2: origin xyz=-0.00201851 -0.0393459 0.00657843 rpy=-1.5708 9.8875e-30 0.474045 -> xyz=-0.0348065 0.0184577 0.00657843 rpy=-1.5708 -1.39143e-17 -1.53308
- joint foot_3: origin xyz=-0.0563458 0.0580779 0.017 rpy=-3.14159 3.67918e-16 -0.349066 -> xyz=-0.0353039 -0.0728116 0.017 rpy=-3.14159 5.33347e-16 1.5708
- joint foot_4: origin xyz=-0.00544005 0.0390203 0.00657843 rpy=1.5708 -1.04558e-16 -0.386778 -> xyz=-0.0348065 -0.0184577 0.00657843 rpy=1.5708 5.47899e-16 1.53308
- joint left_act_shin: origin xyz=0.00337105 0.0348373 -0.005 rpy=-3.14159 3.36129e-15 -1.6057 -> xyz=0.00337105 0.0348373 -0.005 rpy=3.14159 4.11007e-16 -1.6057
- joint left_ankle: origin xyz=-0.03275 0.01025 -0.03505 rpy=2.29827e-15 1.50863e-15 1.5708 -> xyz=-0.03275 0.01025 -0.03505 rpy=1.13027e-31 1.84079e-32 -0.349066
- joint left_foot_frame: origin xyz=-0.0138727 0.005 -0.00631827 rpy=-1.11449e-16 -0.025933 3.14159 -> xyz=-0.0138727 0.005 -0.00631827 rpy=1.76081e-28 -0.025933 -3.14159
- joint left_hip_pitch: origin xyz=-0.03275 0.01025 -0.03505 rpy=-1.67045e-31 1.10934e-31 -0.523599 -> xyz=-0.03275 0.01025 -0.03505 rpy=4.17295e-33 -2.46519e-32 -0.523599
- joint left_hip_roll: limit lower=-0.174533 upper=0.436332 effort=10 velocity=10 -> lower=-0.261799 upper=0.436332 effort=10 velocity=10; origin xyz=0.01905 2.13718e-15 -0.046015 rpy=-1.5708 2.10942e-15 1.5708 -> xyz=0.01905 -6.93889e-18 -0.046015 rpy=-1.5708 6.47552e-16 1.5708
- joint left_hip_yaw: limit lower=-0.349066 upper=0.226893 effort=10 velocity=10 -> lower=-0.349066 upper=0.261799 effort=10 velocity=10; origin xyz=-0.03275 -0.01025 -0.03505 rpy=1.22125e-15 -3.35143e-29 3.14159 -> xyz=-0.03275 -0.01025 -0.03505 rpy=2.3684e-15 1.08579e-16 3.14159
- joint left_knee: limit lower=-1.0472 upper=0.523599 effort=10 velocity=10 -> lower=-1.22173 upper=0.698132 effort=10 velocity=10; origin xyz=0.0340323 -0.0044073 -0.03505 rpy=-3.90287e-16 -1.12803e-15 -2.44346 -> xyz=0.0340323 -0.0044073 -0.03505 rpy=-5.32681e-30 1.15005e-29 -2.44346
- joint leg_act_left: origin xyz=-0.00580147 -0.0504366 -0.006 rpy=3.14159 2.54608e-16 -1.5708 -> xyz=-0.00580147 -0.0504366 -0.006 rpy=3.14159 2.30296e-30 -1.5708
- joint leg_act_right: origin xyz=0.0407786 0.0302425 -0.006 rpy=3.14159 4.90891e-16 -2.51327 -> xyz=-0.00580147 0.0504366 -0.006 rpy=3.14159 5.49001e-16 1.5708
- joint right_ankle: origin xyz=-0.03275 0.01025 -0.03505 rpy=3.71188e-17 -5.56319e-17 -1.5708 -> xyz=-0.03275 0.01025 -0.03505 rpy=8.30013e-32 -1.03288e-31 0.349066
- joint right_foot_frame: origin xyz=-0.0138727 -0.005 -0.00631827 rpy=-4.04466e-32 -0.025933 -3.14159 -> xyz=-0.0138727 -0.005 -0.00631827 rpy=-4.06652e-31 -0.025933 -3.14159
- joint right_hip_pitch: origin xyz=-0.03275 0.01025 -0.03505 rpy=1.95622e-15 3.07394e-15 1.5708 -> xyz=-0.03275 0.01025 -0.03505 rpy=2.64695e-33 -3.38964e-32 0.523599
- joint right_hip_roll: limit lower=-0.523599 upper=0.174533 effort=10 velocity=10 -> lower=-0.436332 upper=0.261799 effort=10 velocity=10; origin xyz=0.01905 -2.77556e-17 -0.046015 rpy=-1.5708 5.52966e-16 1.5708 -> xyz=0.01905 -2.77556e-17 -0.046015 rpy=-1.5708 -8.04717e-18 1.5708
- joint right_hip_yaw: origin xyz=-0.0331099 0.0103599 -0.03505 rpy=2.1982e-15 2.99216e-16 3.14159 -> xyz=-0.0331099 0.0103599 -0.03505 rpy=1.84353e-15 2.057e-16 -3.14159
- joint right_knee: limit lower=-1.0472 upper=0.523599 effort=10 velocity=10 -> lower=-0.698132 upper=1.22173 effort=10 velocity=10; origin xyz=-0.03275 -0.01025 -0.03505 rpy=1.9419e-17 -1.83607e-15 1.5708 -> xyz=0.0340323 0.0044073 -0.03505 rpy=-5.08906e-17 6.93358e-17 2.44346
- joint right_knee_act: origin xyz=-0.0221931 0.0325793 -0.005 rpy=3.14159 -1.40772e-31 -0.488692 -> xyz=-0.0171179 -0.0355095 -0.005 rpy=3.14159 -1.26955e-16 1.6057
- joint tail: limit lower=-0.261799 upper=0.261799 effort=10 velocity=10 -> lower=-0.349066 upper=0.349066 effort=10 velocity=10

Commit message: new urdf + blender dino support

File: awd/data/assets/dino/dino.urdf (robot description, URDF)
Before this commit: robot eyecandy, 54 links, 53 joints
Links:
- link actuator: geometry collision mesh filename=./assets/actuator_convex.stl; visual mesh filename=./assets/actuator.stl
- link actuator_10: geometry collision mesh filename=./assets/actuator_convex.stl; visual mesh filename=./assets/actuator.stl
- link actuator_11: geometry collision mesh filename=./assets/actuator_convex.stl; visual mesh filename=./assets/actuator.stl
- link actuator_12: geometry collision mesh filename=./assets/actuator_convex.stl; visual mesh filename=./assets/actuator.stl
- link actuator_2: geometry collision mesh filename=./assets/actuator_convex.stl; visual mesh filename=./assets/actuator.stl
- link actuator_3: geometry collision mesh filename=./assets/actuator_convex.stl; visual mesh filename=./assets/actuator.stl
- link actuator_4: geometry collision mesh filename=./assets/actuator_convex.stl; visual mesh filename=./assets/actuator.stl
- link actuator_5: geometry collision mesh filename=./assets/actuator_convex.stl; visual mesh filename=./assets/actuator.stl
- link actuator_6: geometry collision mesh filename=./assets/actuator_convex.stl; visual mesh filename=./assets/actuator.stl
- link actuator_7: geometry collision mesh filename=./assets/actuator_convex.stl; visual mesh filename=./assets/actuator.stl
- link actuator_8: geometry collision mesh filename=./assets/actuator_convex.stl; visual mesh filename=./assets/actuator.stl
- link actuator_9: geometry collision mesh filename=./assets/actuator_convex.stl; visual mesh filename=./assets/actuator.stl
- link base: geometry collision mesh filename=./assets/base_convex.stl; visual mesh filename=./assets/base.stl
- link body_back: mass 0.310516 -> 0.33311; geometry collision mesh filename=./assets/body_back_convex.stl; visual mesh filename=./assets/body_back.stl
- link body_electronix_cover: geometry collision mesh filename=./assets/body_electronix_cover_convex.stl; visual mesh filename=./assets/body_electronix_cover.stl
- link body_front: mass 0.153978 -> 0.198161; geometry collision mesh filename=./assets/body_front_convex.stl; visual mesh filename=./assets/body_front.stl
- link box: geometry collision mesh filename=./assets/box_convex.stl; visual mesh filename=./assets/box.stl
- link front_tail: geometry collision mesh filename=./assets/front_tail_convex.stl; visual mesh filename=./assets/front_tail.stl
- link head_attachment: geometry collision mesh filename=./assets/head_attachment_convex.stl; visual mesh filename=./assets/head_attachment.stl
- link head_attachment_2: geometry collision mesh filename=./assets/head_attachment__2_convex.stl; visual mesh filename=./assets/head_attachment__2.stl
- link headdown: mass 0.135224 -> 0.18132; geometry collision mesh filename=./assets/headdown_convex.stl; visual mesh filename=./assets/headdown.stl
- link headup: mass 0.025758 -> 0.0377868; geometry collision mesh filename=./assets/headup_convex.stl; visual mesh filename=./assets/headup.stl
- link hind_tail: geometry collision mesh filename=./assets/hind_tail_convex.stl; visual mesh filename=./assets/hind_tail.stl
- link hip_actuator: geometry collision mesh filename=./assets/hip_actuator_convex.stl; visual mesh filename=./assets/hip_actuator.stl
- link hip_actuator_2: geometry collision mesh filename=./assets/hip_actuator_convex.stl; visual mesh filename=./assets/hip_actuator.stl
- link left_foot_ankle: geometry collision mesh filename=./assets/left_foot_ankle_convex.stl; visual mesh filename=./assets/left_foot_ankle.stl
- link left_foot_cover: geometry collision mesh filename=./assets/left_foot_cover_convex.stl; visual mesh filename=./assets/left_foot_cover.stl
- link left_foot_tpu: mass 0.042081 -> 0.0478193; geometry collision mesh filename=./assets/left_foot_tpu_convex.stl; visual mesh filename=./assets/left_foot_tpu.stl
- link left_leg_shin: geometry collision mesh filename=./assets/left_leg_shin_convex.stl; visual mesh filename=./assets/left_leg_shin.stl
- link left_motor_thigh: geometry collision mesh filename=./assets/left_motor_thigh_convex.stl; visual mesh filename=./assets/left_motor_thigh.stl
- link left_roll_to_pitch: geometry collision mesh filename=./assets/left_roll_to_pitch_convex.stl; visual mesh filename=./assets/left_roll_to_pitch.stl
- link left_upper_cover: mass 0.24609 -> 0.243001; geometry collision mesh filename=./assets/left_upper_cover_convex.stl; visual mesh filename=./assets/left_upper_cover.stl
- link liion: geometry collision mesh filename=./assets/liion_convex.stl; visual mesh filename=./assets/liion.stl
- link liion_2: geometry collision mesh filename=./assets/liion_convex.stl; visual mesh filename=./assets/liion.stl
- link motor_driver: geometry collision mesh filename=./assets/motor_driver_convex.stl; visual mesh filename=./assets/motor_driver.stl
- link neck_left: geometry collision mesh filename=./assets/neck_left_convex.stl; visual mesh filename=./assets/neck_left.stl
- link neck_right: geometry collision mesh filename=./assets/neck_right_convex.stl; visual mesh filename=./assets/neck_right.stl
- link powermodule: geometry collision mesh filename=./assets/powermodule_convex.stl; visual mesh filename=./assets/powermodule.stl
- link raspberrypizerow: geometry collision mesh filename=./assets/raspberrypizerow_convex.stl; visual mesh filename=./assets/raspberrypizerow.stl
- link right_foot_ankle: geometry collision mesh filename=./assets/right_foot_ankle_convex.stl; visual mesh filename=./assets/right_foot_ankle.stl
- link right_foot_cover: geometry collision mesh filename=./assets/right_foot_cover_convex.stl; visual mesh filename=./assets/right_foot_cover.stl
- link right_foot_tpu: mass 0.042081 -> 0.0478193; geometry collision mesh filename=./assets/right_foot_tpu_convex.stl; visual mesh filename=./assets/right_foot_tpu.stl
- link right_leg_shin: geometry collision mesh filename=./assets/right_leg_shin_convex.stl; visual mesh filename=./assets/right_leg_shin.stl
- link right_leg_thigh: geometry collision mesh filename=./assets/right_leg_thigh_convex.stl; visual mesh filename=./assets/right_leg_thigh.stl
- link right_roll_to_pitch: mass 0.059066 -> 0.0527166; geometry collision mesh filename=./assets/right_roll_to_pitch_convex.stl; visual mesh filename=./assets/right_roll_to_pitch.stl
- link right_upper_cover: mass 0.24609 -> 0.243001; geometry collision mesh filename=./assets/right_upper_cover_convex.stl; visual mesh filename=./assets/right_upper_cover.stl
- link roll_bearing: geometry collision mesh filename=./assets/roll_bearing_convex.stl; visual mesh filename=./assets/roll_bearing.stl
- link roll_bearing_2: geometry collision mesh filename=./assets/roll_bearing_convex.stl; visual mesh filename=./assets/roll_bearing.stl
- link tail_connector: geometry collision mesh filename=./assets/tail_connector_convex.stl; visual mesh filename=./assets/tail_connector.stl
- link trunk_top: geometry collision mesh filename=./assets/trunk_top_convex.stl; visual mesh filename=./assets/trunk_top.stl
Joints:
- joint act_in_hip_left: origin xyz=0.0523698 0.01025 0.00236 rpy=3.14159 1.5708 0 -> xyz=0.0523698 0.01025 0.00236 rpy=-3.14159 1.5708 0
- joint act_in_hip_right: origin xyz=-0.0523698 -0.01025 0.00236 rpy=-1.80411e-16 1.5708 0 -> xyz=-0.0523698 -0.01025 0.00236 rpy=-5.55112e-17 1.5708 0
- joint act_in_neck_left: origin xyz=0.033 -0.01025 0.002425 rpy=3.14159 1.25677e-56 -6.22302e-61 -> xyz=0.033 -0.01025 0.002425 rpy=-3.14159 -1.21805e-31 -6.16298e-32
- joint act_in_neck_right: origin xyz=-0.00375 -0.0205 -0.032 rpy=1.33227e-15 -3.42591e-23 2.20635e-30 -> xyz=-0.00375 -0.0205 -0.032 rpy=3.19795e-17 -1.94613e-17 -3.26638e-30
- joint body_back: child body_back -> body_front
- joint body_front: child body_front -> body_back; origin xyz=0.0041479 0.01 -0.009 rpy=3.14159 1.53384 -2.37255e-31 -> xyz=-0.0048521 0.01 -0.0082 rpy=-2.16068e-17 1.53384 -2.06118e-15; parent body_back -> body_front
- joint cover_to_leg_left: origin xyz=-0.007 -0.02 -0.01 rpy=-6.58031e-17 -6.41721e-17 -2.30383 -> xyz=-0.007 -0.02 -0.01 rpy=7.55956e-15 1.64177e-15 -2.30383
- joint cover_to_leg_right: origin xyz=-0.007 0.02 -0.01 rpy=1.73993e-16 5.2061e-16 2.35619 -> xyz=-0.007 0.02 -0.01 rpy=6.98868e-16 -1.19452e-16 2.35619
- joint dino_head: origin xyz=-1.38778e-17 -0.00975 -0.008 rpy=-2.60399e-26 -6.18763e-30 3.97644e-28 -> xyz=-1.38778e-17 -0.00975 -0.008 rpy=-5.71924e-29 4.11754e-17 -1.31976e-15
- joint dino_head_w_act: origin xyz=-0.03275 0.01025 -0.03505 rpy=-2.1896e-27 1.26218e-29 -3.14159 -> xyz=-0.03275 0.01025 -0.03505 rpy=3.06867e-28 6.31089e-30 -3.14159
- joint foot_1: origin xyz=-0.0256494 0.0333834 0.017 rpy=-3.14159 1.11474e-15 -1.5708 -> xyz=-0.0256494 0.0333834 0.017 rpy=3.14159 5.81694e-16 -1.5708
- joint foot_2: origin xyz=-0.0348065 0.0184577 0.00657843 rpy=-1.5708 -1.39143e-17 -1.53308 -> xyz=-0.0348065 0.0184577 0.00657843 rpy=-1.5708 -1.78275e-16 -1.53308
- joint foot_3: origin xyz=-0.0353039 -0.0728116 0.017 rpy=-3.14159 5.33347e-16 1.5708 -> xyz=-0.0353039 -0.0728116 0.017 rpy=-3.14159 -1.22683e-16 1.5708
- joint foot_4: origin xyz=-0.0348065 -0.0184577 0.00657843 rpy=1.5708 5.47899e-16 1.53308 -> xyz=-0.0348065 -0.0184577 0.00657843 rpy=1.5708 1.09067e-17 1.53308
- joint head: origin xyz=0.0300601 0.0512 0.0230859 rpy=-3.14159 -0.121002 -3.14159 -> xyz=0.0213775 0.0551 0.0224423 rpy=-3.14159 -0.121002 -3.14159
- joint head_pitch: origin xyz=0.029 -0.01025 -0.0338 rpy=1.30346e-23 1.27104e-15 -1.5708 -> xyz=0.029 -0.01025 -0.0338 rpy=1.2091e-16 -6.8789e-17 -1.5708
- joint head_yaw: origin xyz=0.00369936 0.025 0.01845 rpy=1.5708 4.34139e-39 0 -> xyz=0.00369936 0.025 0.01845 rpy=1.5708 2.86854e-32 0
- joint hind_tail: origin xyz=0.0645127 -4.72364e-06 0.000584758 rpy=3.7929e-16 0.268289 -1.25764e-15 -> xyz=0.0645127 -4.72364e-06 0.000584758 rpy=2.08843e-15 0.268289 -4.38561e-15
- joint left_act_shin: origin xyz=0.00337105 0.0348373 -0.005 rpy=3.14159 4.11007e-16 -1.6057 -> xyz=0.00337105 0.0348373 -0.005 rpy=-3.14159 -1.07809e-15 -1.6057
- joint left_ankle: origin xyz=-0.03275 0.01025 -0.03505 rpy=1.13027e-31 1.84079e-32 -0.349066 -> xyz=-0.03275 0.01025 -0.03505 rpy=-1.30487e-31 -1.82467e-32 -0.349066
- joint left_foot_frame: origin xyz=-0.0138727 0.005 -0.00631827 rpy=1.76081e-28 -0.025933 -3.14159 -> xyz=-0.0138727 0.005 -0.00631827 rpy=-1.37154e-14 -0.025933 3.14159
- joint left_hip_pitch: origin xyz=-0.03275 0.01025 -0.03505 rpy=4.17295e-33 -2.46519e-32 -0.523599 -> xyz=-0.03275 0.01025 -0.03505 rpy=-3.95057e-33 -9.24446e-32 -0.523599
- joint left_hip_roll: origin xyz=0.01905 -6.93889e-18 -0.046015 rpy=-1.5708 6.47552e-16 1.5708 -> xyz=0.01905 1.04083e-17 -0.046015 rpy=-1.5708 -5.55112e-17 1.5708
- joint left_hip_yaw: origin xyz=-0.03275 -0.01025 -0.03505 rpy=2.3684e-15 1.08579e-16 3.14159 -> xyz=-0.03275 -0.01025 -0.03505 rpy=1.66533e-15 1.66533e-16 -3.14159
- joint left_knee: origin xyz=0.0340323 -0.0044073 -0.03505 rpy=-5.32681e-30 1.15005e-29 -2.44346 -> xyz=0.0340323 -0.0044073 -0.03505 rpy=9.55429e-15 -1.58817e-15 -2.44346
- joint leg_act_left: origin xyz=-0.00580147 -0.0504366 -0.006 rpy=3.14159 2.30296e-30 -1.5708 -> xyz=-0.00580147 -0.0504366 -0.006 rpy=-3.14159 -4.13619e-15 -1.5708
- joint leg_act_right: origin xyz=-0.00580147 0.0504366 -0.006 rpy=3.14159 5.49001e-16 1.5708 -> xyz=-0.00580147 0.0504366 -0.006 rpy=-3.14159 5.58679e-16 1.5708
- joint lid: origin xyz=-0.0390284 0.035 0.148456 rpy=3.14159 0.0586009 -6.61486e-34 -> xyz=-0.16958 0.025 -0.0373289 rpy=3.14159 -1.47524 1.95595e-23
- joint neck_pitch: limit lower=-1.0472 upper=1.5708 effort=10 velocity=10 -> lower=-1.0472 upper=0.261799 effort=10 velocity=10; origin xyz=0.03275 -0.01025 -0.03505 rpy=5.68022e-31 6.13832e-30 1.5708 -> xyz=0.03275 -0.01025 -0.03505 rpy=1.27148e-15 2.16678e-15 1.5708
- joint right_ankle: origin xyz=-0.03275 0.01025 -0.03505 rpy=8.30013e-32 -1.03288e-31 0.349066 -> xyz=-0.03275 0.01025 -0.03505 rpy=-9.00623e-32 3.54234e-33 0.349066
- joint right_foot_frame: origin xyz=-0.0138727 -0.005 -0.00631827 rpy=-4.06652e-31 -0.025933 -3.14159 -> xyz=-0.0138727 -0.005 -0.00631827 rpy=3.71266e-16 -0.025933 -3.14159
- joint right_hip_pitch: origin xyz=-0.03275 0.01025 -0.03505 rpy=2.64695e-33 -3.38964e-32 0.523599 -> xyz=-0.03275 0.01025 -0.03505 rpy=-1.01993e-31 6.16298e-32 0.523599
- joint right_hip_roll: origin xyz=0.01905 -2.77556e-17 -0.046015 rpy=-1.5708 -8.04717e-18 1.5708 -> xyz=0.01905 -2.46678e-15 -0.046015 rpy=-1.5708 -6.88059e-16 1.5708
- joint right_hip_yaw: origin xyz=-0.0331099 0.0103599 -0.03505 rpy=1.84353e-15 2.057e-16 -3.14159 -> xyz=-0.0331099 0.0103599 -0.03505 rpy=1.84353e-15 1.44468e-16 3.14159
- joint right_knee: origin xyz=0.0340323 0.0044073 -0.03505 rpy=-5.08906e-17 6.93358e-17 2.44346 -> xyz=0.0340323 0.0044073 -0.03505 rpy=2.70465e-16 1.25637e-16 2.44346
- joint right_knee_act: origin xyz=-0.0171179 -0.0355095 -0.005 rpy=3.14159 -1.26955e-16 1.6057 -> xyz=-0.0171179 -0.0355095 -0.005 rpy=3.14159 -1.97425e-16 1.6057
- joint tail: origin xyz=-0.03275 -0.01025 -0.03505 rpy=9.46854e-17 -4.22346e-17 -3.14159 -> xyz=-0.03275 -0.01025 -0.03505 rpy=-4.06308e-17 2.8936e-16 3.14159
- joint tail_holder: origin xyz=0.0580257 -3.94149e-06 -0.0229936 rpy=-1.37852e-16 0.174533 8.46988e-30 -> xyz=0.0580257 -3.94149e-06 -0.0229936 rpy=3.95912e-17 0.174533 6.21269e-17
