Commit message: new urdf + mjf

File: awd/data/assets/dino/dino.urdf (robot description, URDF)
Before this commit: robot eyecandy, 54 links, 53 joints
Links:
- link actuator: geometry collision mesh filename=./assets/actuator_convex.stl; visual mesh filename=./assets/actuator.stl
- link actuator_10: geometry collision mesh filename=./assets/actuator_convex.stl; visual mesh filename=./assets/actuator.stl
- link actuator_11: geometry collision mesh filename=./assets/actuator_convex.stl; visual mesh filename=./assets/actuator.stl
- link actuator_12: geometry collision mesh filename=./assets/actuator_convex.stl; visual mesh filename=./assets/actuator.stl
- link actuator_2: geometry collision mesh filename=./assets/actuator_convex.stl; visual mesh filename=./assets/actuator.stl
- link actuator_3: geometry collision mesh filename=./assets/actuator_convex.stl; visual mesh filename=./assets/actuator.stl
- link actuator_4: geometry collision mesh filename=./assets/actuator_convex.stl; visual mesh filename=./assets/actuator.stl
- link actuator_5: geometry collision mesh filename=./assets/actuator_convex.stl; visual mesh filename=./assets/actuator.stl
- link actuator_6: geometry collision mesh filename=./assets/actuator_convex.stl; visual mesh filename=./assets/actuator.stl
- link actuator_7: geometry collision mesh filename=./assets/actuator_convex.stl; visual mesh filename=./assets/actuator.stl
- link actuator_8: geometry collision mesh filename=./assets/actuator_convex.stl; visual mesh filename=./assets/actuator.stl
- link actuator_9: geometry collision mesh filename=./assets/actuator_convex.stl; visual mesh filename=./assets/actuator.stl
- link base: geometry collision mesh filename=./assets/base_convex.stl; visual mesh filename=./assets/base.stl
- link body_back: geometry collision mesh filename=./assets/body_back_convex.stl; visual mesh filename=./assets/body_back.stl
- link body_electronix_cover: geometry collision mesh filename=./assets/body_electronix_cover_convex.stl; visual mesh filename=./assets/body_electronix_cover.stl
- link body_front: geometry collision mesh filename=./assets/body_front_convex.stl; visual mesh filename=./assets/body_front.stl
- link box: geometry collision mesh filename=./assets/box_convex.stl; visual mesh filename=./assets/box.stl
- link front_tail: geometry collision mesh filename=./assets/front_tail_convex.stl; visual mesh filename=./assets/front_tail.stl
- link head_attachment: geometry collision mesh filename=./assets/head_attachment_convex.stl; visual mesh filename=./assets/head_attachment.stl
- link head_attachment_2: geometry collision mesh filename=./assets/head_attachment__2_convex.stl; visual mesh filename=./assets/head_attachment__2.stl
- link headdown: mass 0.202458 -> 0.18132; geometry collision mesh filename=./assets/headdown_convex.stl; visual mesh filename=./assets/headdown.stl
- link headup: geometry collision mesh filename=./assets/headup_convex.stl; visual mesh filename=./assets/headup.stl
- link hind_tail: geometry collision mesh filename=./assets/hind_tail_convex.stl; visual mesh filename=./assets/hind_tail.stl
- link hip_actuator: geometry collision mesh filename=./assets/hip_actuator_convex.stl; visual mesh filename=./assets/hip_actuator.stl
- link hip_actuator_2: geometry collision mesh filename=./assets/hip_actuator_convex.stl; visual mesh filename=./assets/hip_actuator.stl
- link left_foot_ankle: geometry collision mesh filename=./assets/left_foot_ankle_convex.stl; visual mesh filename=./assets/left_foot_ankle.stl
- link left_foot_cover: geometry collision mesh filename=./assets/left_foot_cover_convex.stl; visual mesh filename=./assets/left_foot_cover.stl
- link left_foot_tpu: geometry collision mesh filename=./assets/left_foot_tpu_convex.stl; visual mesh filename=./assets/left_foot_tpu.stl
- link left_leg_shin: geometry collision mesh filename=./assets/left_leg_shin_convex.stl; visual mesh filename=./assets/left_leg_shin.stl
- link left_motor_thigh: geometry collision mesh filename=./assets/left_motor_thigh_convex.stl; visual mesh filename=./assets/left_motor_thigh.stl
- link left_roll_to_pitch: geometry collision mesh filename=./assets/left_roll_to_pitch_convex.stl; visual mesh filename=./assets/left_roll_to_pitch.stl
- link left_upper_cover: geometry collision mesh filename=./assets/left_upper_cover_convex.stl; visual mesh filename=./assets/left_upper_cover.stl
- link liion: geometry collision mesh filename=./assets/liion_convex.stl; visual mesh filename=./assets/liion.stl
- link liion_2: geometry collision mesh filename=./assets/liion_convex.stl; visual mesh filename=./assets/liion.stl
- link motor_driver: geometry collision mesh filename=./assets/motor_driver_convex.stl; visual mesh filename=./assets/motor_driver.stl
- link neck_left: geometry collision mesh filename=./assets/neck_left_convex.stl; visual mesh filename=./assets/neck_left.stl
- link neck_right: geometry collision mesh filename=./assets/neck_right_convex.stl; visual mesh filename=./assets/neck_right.stl
- link powermodule: geometry collision mesh filename=./assets/powermodule_convex.stl; visual mesh filename=./assets/powermodule.stl
- link raspberrypizerow: geometry collision mesh filename=./assets/raspberrypizerow_convex.stl; visual mesh filename=./assets/raspberrypizerow.stl
- link right_foot_ankle: geometry collision mesh filename=./assets/right_foot_ankle_convex.stl; visual mesh filename=./assets/right_foot_ankle.stl
- link right_foot_cover: geometry collision mesh filename=./assets/right_foot_cover_convex.stl; visual mesh filename=./assets/right_foot_cover.stl
- link right_foot_tpu: geometry collision mesh filename=./assets/right_foot_tpu_convex.stl; visual mesh filename=./assets/right_foot_tpu.stl
- link right_leg_shin: geometry collision mesh filename=./assets/right_leg_shin_convex.stl; visual mesh filename=./assets/right_leg_shin.stl
- link right_leg_thigh: geometry collision mesh filename=./assets/right_leg_thigh_convex.stl; visual mesh filename=./assets/right_leg_thigh.stl
- link right_roll_to_pitch: geometry collision mesh filename=./assets/right_roll_to_pitch_convex.stl; visual mesh filename=./assets/right_roll_to_pitch.stl
- link right_upper_cover: geometry collision mesh filename=./assets/right_upper_cover_convex.stl; visual mesh filename=./assets/right_upper_cover.stl
- link roll_bearing: geometry collision mesh filename=./assets/roll_bearing_convex.stl; visual mesh filename=./assets/roll_bearing.stl
- link roll_bearing_2: geometry collision mesh filename=./assets/roll_bearing_convex.stl; visual mesh filename=./assets/roll_bearing.stl
- link tail_connector: geometry collision mesh filename=./assets/tail_connector_convex.stl; visual mesh filename=./assets/tail_connector.stl
- link trunk_top: geometry collision mesh filename=./assets/trunk_top_convex.stl; visual mesh filename=./assets/trunk_top.stl
Joints:
- joint act_in_hip_right: origin xyz=-0.0523698 -0.01025 0.00236 rpy=1.57772e-30 1.5708 0 -> xyz=-0.0523698 -0.01025 0.00236 rpy=-5.55112e-17 1.5708 0
- joint act_in_neck_left: origin xyz=0.033 -0.01025 0.002425 rpy=3.14159 -0 0 -> xyz=0.033 -0.01025 0.002425 rpy=-3.14159 -1.21805e-31 -6.16298e-32
- joint act_in_neck_right: origin xyz=-0.00375 -0.0205 -0.032 rpy=-1.39224e-14 -1.12231e-15 1.07149e-28 -> xyz=-0.00375 -0.0205 -0.032 rpy=3.19795e-17 -1.94613e-17 -3.26638e-30
- joint act_to_trunk: origin xyz=-0.00196569 0.0161 -0.02762 rpy=-1.5708 2.98372e-16 -2.79509e-16 -> xyz=-0.00196569 0.0161 -0.02762 rpy=-1.5708 1.66533e-16 -4.18054e-31
- joint batt_one: origin xyz=0.0004 -0.0355 -0.011 rpy=1.5708 5.85194e-16 2.35988e-14 -> xyz=0.0004 -0.0355 -0.011 rpy=1.5708 5.84918e-16 2.08238e-15
- joint batt_two: origin xyz=-0.0196 -0.0355 -0.011 rpy=1.5708 5.87121e-16 1.95542e-15 -> xyz=-0.0196 -0.0355 -0.011 rpy=1.5708 5.84688e-16 2.08531e-15
- joint battpack: origin xyz=-0.0515073 0.0096 0.042 rpy=1.5708 5.00235e-15 1.5708 -> xyz=-0.0515073 0.0096 0.042 rpy=1.5708 9.86076e-32 1.5708
- joint bearing: origin xyz=7.1259e-05 0.02061 0.0278 rpy=-3.14159 -1.5335e-15 3.14159 -> xyz=7.1259e-05 0.02061 0.0278 rpy=-3.14159 -0 -3.14159
- joint body_back: origin xyz=0.0176498 -0.01 1.38778e-16 rpy=-5.00235e-15 7.42462e-16 -3.55832e-20 -> xyz=0.0176498 -0.01 -2.77556e-17 rpy=-9.86076e-32 -3.9443e-31 0
- joint body_front: origin xyz=-0.0048521 0.01 -0.0082 rpy=-6.95631e-17 1.53384 6.44043e-16 -> xyz=-0.0048521 0.01 -0.0082 rpy=-2.16068e-17 1.53384 -2.06118e-15
- joint body_to_base: origin xyz=7.1259e-05 -0.02061 0.0278 rpy=-3.14159 -1.5335e-15 3.14159 -> xyz=7.1259e-05 -0.02061 0.0278 rpy=-3.14159 -0 -3.14159
- joint charger_booster: origin xyz=-0.0598957 0.01936 0.0011 rpy=-2.86244e-17 1.5708 0 -> xyz=-0.0598957 0.01936 0.0011 rpy=-7.49401e-16 1.5708 0
- joint cover_to_leg_left: origin xyz=-0.007 -0.02 -0.01 rpy=4.26605e-15 -1.38261e-15 -2.35619 -> xyz=-0.007 -0.02 -0.01 rpy=7.55956e-15 1.64177e-15 -2.30383
- joint cover_to_leg_right: origin xyz=-0.007 0.02 -0.01 rpy=4.79141e-15 -3.89605e-15 2.35619 -> xyz=-0.007 0.02 -0.01 rpy=6.98868e-16 -1.19452e-16 2.35619
- joint dino_head: origin xyz=-6.93889e-17 -0.00975 -0.008 rpy=5.31994e-15 5.18662e-18 -6.37863e-30 -> xyz=-1.38778e-17 -0.00975 -0.008 rpy=-5.71924e-29 4.11754e-17 -1.31976e-15
- joint dino_head_w_act: origin xyz=-0.03275 0.01025 -0.03505 rpy=-5.2923e-15 2.38336e-15 3.14159 -> xyz=-0.03275 0.01025 -0.03505 rpy=3.06867e-28 6.31089e-30 -3.14159
- joint foot_1: origin xyz=-0.0256494 0.0333834 0.017 rpy=-3.14159 -5.43972e-17 -1.5708 -> xyz=-0.0256494 0.0333834 0.017 rpy=3.14159 5.81694e-16 -1.5708
- joint foot_2: origin xyz=-0.0348065 0.0184577 0.00657843 rpy=-1.5708 1.70885e-18 -1.53308 -> xyz=-0.0348065 0.0184577 0.00657843 rpy=-1.5708 -1.78275e-16 -1.53308
- joint foot_3: origin xyz=-0.0353039 -0.0728116 0.017 rpy=-3.14159 7.6274e-16 1.5708 -> xyz=-0.0353039 -0.0728116 0.017 rpy=-3.14159 -1.22683e-16 1.5708
- joint foot_4: origin xyz=-0.0348065 -0.0184577 0.00657843 rpy=1.5708 2.30866e-18 1.53308 -> xyz=-0.0348065 -0.0184577 0.00657843 rpy=1.5708 1.09067e-17 1.53308
- joint head_pitch: limit lower=-1.00616 upper=1.08823 effort=10 velocity=10 -> lower=-1.0472 upper=1.0472 effort=10 velocity=10; origin xyz=0.029 -0.01025 -0.0338 rpy=1.30202e-16 -2.20411e-15 -1.61183 -> xyz=0.029 -0.01025 -0.0338 rpy=1.2091e-16 -6.8789e-17 -1.5708
- joint head_yaw: origin xyz=0.00369936 0.025 0.01845 rpy=1.5708 -2.02235e-32 1.50603e-18 -> xyz=0.00369936 0.025 0.01845 rpy=1.5708 2.86854e-32 0
- joint hind_tail: origin xyz=0.0645127 -4.72364e-06 0.000584758 rpy=-4.07364e-15 0.268289 8.59453e-15 -> xyz=0.0645127 -4.72364e-06 0.000584758 rpy=2.08843e-15 0.268289 -4.38561e-15
- joint hip_act_trunk_left: origin xyz=-0.0525357 -0.01036 -0.0311 rpy=3.14159 -4.09395e-16 3.14159 -> xyz=-0.0525357 -0.01036 -0.0311 rpy=-3.14159 -1.66533e-16 -3.14159
- joint hip_act_trunk_right: origin xyz=-0.0525357 0.01036 -0.0311 rpy=-3.14159 -5.55112e-16 3.14159 -> xyz=-0.0525357 0.01036 -0.0311 rpy=-3.14159 -1.86117e-16 -3.14159
- joint left_act_shin: origin xyz=0.00337105 0.0348373 -0.005 rpy=-3.14159 -4.31026e-17 -1.6057 -> xyz=0.00337105 0.0348373 -0.005 rpy=-3.14159 -1.07809e-15 -1.6057
- joint left_ankle: origin xyz=-0.03275 0.01025 -0.03505 rpy=3.68296e-31 -1.80943e-30 -0.383972 -> xyz=-0.03275 0.01025 -0.03505 rpy=-1.30487e-31 -1.82467e-32 -0.349066
- joint left_foot_frame: origin xyz=-0.0138727 0.005 -0.00631827 rpy=-2.25568e-28 -0.025933 -3.14159 -> xyz=-0.0138727 0.005 -0.00631827 rpy=-1.37154e-14 -0.025933 3.14159
- joint left_hip_pitch: origin xyz=-0.03275 0.01025 -0.03505 rpy=-1.37063e-30 -6.25343e-32 -0.523599 -> xyz=-0.03275 0.01025 -0.03505 rpy=-3.95057e-33 -9.24446e-32 -0.523599
- joint left_hip_roll: origin xyz=0.01905 -3.46945e-18 -0.046015 rpy=-1.5708 -1.46516e-29 1.5708 -> xyz=0.01905 1.04083e-17 -0.046015 rpy=-1.5708 -5.55112e-17 1.5708
- joint left_hip_yaw: origin xyz=-0.03275 -0.01025 -0.03505 rpy=-9.15416e-15 -1.21801e-16 -3.14159 -> xyz=-0.03275 -0.01025 -0.03505 rpy=1.66533e-15 1.66533e-16 -3.14159
- joint left_knee: origin xyz=0.0340323 -0.0044073 -0.03505 rpy=-3.23833e-28 -6.71832e-28 -2.44346 -> xyz=0.0340323 -0.0044073 -0.03505 rpy=9.55429e-15 -1.58817e-15 -2.44346
- joint leg_act_left: origin xyz=-0.00580147 -0.0504366 -0.006 rpy=3.14159 1.8444e-28 -1.5708 -> xyz=-0.00580147 -0.0504366 -0.006 rpy=-3.14159 -4.13619e-15 -1.5708
- joint leg_act_right: origin xyz=-0.00580147 0.0504366 -0.006 rpy=-3.14159 -1.13706e-28 1.5708 -> xyz=-0.00580147 0.0504366 -0.006 rpy=-3.14159 5.58679e-16 1.5708
- joint lid: origin xyz=-0.16958 0.025 -0.0373289 rpy=-3.14159 -1.47524 -5.30016e-15 -> xyz=-0.16958 0.025 -0.0373289 rpy=3.14159 -1.47524 1.95595e-23
- joint mpu_frame: origin xyz=0.0031102 0.010157 -0.0369 rpy=-1.5708 5.75928e-16 2.77949e-17 -> xyz=0.0031102 0.010157 -0.0369 rpy=-1.5708 2.60786e-16 -4.18054e-31
- joint neck_pitch: origin xyz=0.03275 -0.01025 -0.03505 rpy=-1.41405e-16 4.51939e-15 1.5708 -> xyz=0.03275 -0.01025 -0.03505 rpy=1.27148e-15 2.16678e-15 1.5708
- joint right_ankle: origin xyz=-0.03275 0.01025 -0.03505 rpy=3.3116e-31 1.96116e-30 0.383972 -> xyz=-0.03275 0.01025 -0.03505 rpy=-9.00623e-32 3.54234e-33 0.349066
- joint right_foot_frame: origin xyz=-0.0138727 -0.005 -0.00631827 rpy=1.70264e-29 -0.025933 -3.14159 -> xyz=-0.0138727 -0.005 -0.00631827 rpy=3.71266e-16 -0.025933 -3.14159
- joint right_hip_pitch: origin xyz=-0.03275 0.01025 -0.03505 rpy=1.0813e-30 1.33934e-31 0.523599 -> xyz=-0.03275 0.01025 -0.03505 rpy=-1.01993e-31 6.16298e-32 0.523599
- joint right_hip_roll: origin xyz=0.01905 1.38778e-17 -0.046015 rpy=-1.5708 -3.47657e-28 1.5708 -> xyz=0.01905 -2.46678e-15 -0.046015 rpy=-1.5708 -6.88059e-16 1.5708
- joint right_hip_yaw: origin xyz=-0.0331099 0.0103599 -0.03505 rpy=1.4039e-14 -4.42558e-17 3.14159 -> xyz=-0.0331099 0.0103599 -0.03505 rpy=1.84353e-15 1.44468e-16 3.14159
- joint right_knee: origin xyz=0.0340323 0.0044073 -0.03505 rpy=7.0087e-16 -7.64176e-16 2.44346 -> xyz=0.0340323 0.0044073 -0.03505 rpy=2.70465e-16 1.25637e-16 2.44346
- joint right_knee_act: origin xyz=-0.0171179 -0.0355095 -0.005 rpy=3.14159 1.24719e-27 1.6057 -> xyz=-0.0171179 -0.0355095 -0.005 rpy=3.14159 -1.97425e-16 1.6057
- joint rpi: origin xyz=-0.0822857 0.0115 -0.0379 rpy=-2.72803e-15 5.41234e-16 -6.95838e-17 -> xyz=-0.0822857 0.0115 -0.0379 rpy=-2.33147e-15 2.60786e-16 -8.04893e-31
- joint servo_driver: origin xyz=-0.0628957 -0.01976 -0.0294 rpy=-1.5708 -9.45213e-18 -1.5708 -> xyz=-0.0628957 -0.01976 -0.0294 rpy=-1.5708 -1.16573e-15 -1.5708
- joint tail: limit lower=-0.20689 upper=0.491242 effort=10 velocity=10 -> lower=-0.349066 upper=0.349066 effort=10 velocity=10; origin xyz=-0.03275 -0.01025 -0.03505 rpy=1.03287e-14 1.59777e-15 2.99942 -> xyz=-0.03275 -0.01025 -0.03505 rpy=-4.06308e-17 2.8936e-16 3.14159
- joint tail_holder: origin xyz=0.0580257 -3.94149e-06 -0.0229936 rpy=-1.89315e-15 0.174533 6.69187e-17 -> xyz=0.0580257 -3.94149e-06 -0.0229936 rpy=3.95912e-17 0.174533 6.21269e-17
- joint top_to_bottom_trunk: origin xyz=0.0198569 -2.57957e-17 0.103675 rpy=3.14159 7.42462e-16 -3.55832e-20 -> xyz=0.0198569 -1.78403e-17 0.103675 rpy=3.14159 -3.9443e-31 0
- joint trunk_act_hip: origin xyz=-0.0693357 0.01025 0.0003 rpy=4.55382e-15 8.18789e-16 3.77495e-16 -> xyz=-0.0693357 0.01025 0.0003 rpy=1.55095e-16 8.36883e-28 2.96596e-27
- joint trunk_frame: origin xyz=-0.008 -5.21437e-16 0.0025 rpy=-5.05312e-15 3.33067e-16 2.77302e-16 -> xyz=-0.008 -5.20417e-18 0.0025 rpy=-8.07794e-28 -1.61559e-27 1.88168e-27

Commit message: dino

File: awd/data/assets/dino/dino.urdf (robot description, URDF)
Before this commit: robot eyecandy, 54 links, 53 joints
Joints:
- joint hind_tail: limit lower=-0.698132 upper=0.698132 effort=10 velocity=10 -> effort=10 velocity=10; type revolute -> fixed
